File: kiban/mother-ring-02/mother-ring-02.kicad_sch (KiCad schematic)
At the start: 24 parts, among them J1 LED01, J10 CHARGE, J11 POWER, J12 5V, J13 3V3, J14 BATTERY, J15 POWER, J2 LED02, J3 LED03, J4 LED04, J5 LED05, J6 POWER-01, J7 POWER-02, J8 ESP32-01, J9 ESP32-01

Commit message: kiban: mother-ring board update + v02/v03 iterations
Connections:
- net GND: no longer J14.1 (Pin_1), J7.4 (Pin_4), J8.5 (Pin_5)
- net P+: now also J14.1 (Pin_1), J7.4 (Pin_4); no longer J14.3 (Pin_3), J7.6 (Pin_6)
- new net GPIO08: J8.5 (Pin_5)
- new net P-: J14.3 (Pin_3), J7.6 (Pin_6)
