File: kiban/mother-ring-03/mother-ring-03.kicad_pcb (KiCad board)
At the start: 2 copper layers, 88 x 88 mm, 26 parts, among them J1 LED01, J10 CHARGE, J11 POWER, J12 5V, J13 3V3, J14 BATTERY, J15 POWER, J2 LED02, J3 LED03, J4 LED04, J5 LED05, J6 POWER-01, J7 POWER-02, J8 ESP32-01, J9 ESP32-01

Commit message: kiban: mother-ring board update + v02/v03 iterations
Other:
- outline, holes or cut-outs redrawn
Changed lines of the file:
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@@
 		(property ki_fp_filters "Connector*:*_1x??_*")
 		(sheetname "/")
-		(sheetfile "mother-ring.kicad_sch")
+		(sheetfile "mother-ring-03.kicad_sch")
 		(units
 			(unit
@@
 		(property ki_fp_filters "Connector*:*_1x??_*")
 		(sheetname "/")
-		(sheetfile "mother-ring.kicad_sch")
+		(sheetfile "mother-ring-03.kicad_sch")
 		(units
 			(unit
@@
 		(property ki_fp_filters "Connector*:*_1x??_*")
 		(sheetname "/")
-		(sheetfile "mother-ring.kicad_sch")
+		(sheetfile "mother-ring-03.kicad_sch")
 		(units
 			(unit
@@
 		(property ki_fp_filters "Connector*:*_1x??_*")
 		(sheetname "/")
-		(sheetfile "mother-ring.kicad_sch")
+		(sheetfile "mother-ring-03.kicad_sch")
 		(units
 			(unit
@@
 		(property ki_fp_filters "C_*")
 		(sheetname "/")
-		(sheetfile "mother-ring.kicad_sch")
+		(sheetfile "mother-ring-03.kicad_sch")
 		(units
 			(unit
@@
 		(property ki_fp_filters "Connector*:*_1x??_*")
 		(sheetname "/")
-		(sheetfile "mother-ring.kicad_sch")
+		(sheetfile "mother-ring-03.kicad_sch")
 		(units
 			(unit
@@
 		(property ki_fp_filters "R_*")
 		(sheetname "/")
-		(sheetfile "mother-ring.kicad_sch")
+		(sheetfile "mother-ring-03.kicad_sch")
 		(units
 			(unit
@@
 		(property ki_fp_filters "Connector*:*_1x??_*")
 		(sheetname "/")
-		(sheetfile "mother-ring.kicad_sch")
+		(sheetfile "mother-ring-03.kicad_sch")
 		(units
 			(unit
@@
 		(property ki_fp_filters "R_*")
 		(sheetname "/")
-		(sheetfile "mother-ring.kicad_sch")
+		(sheetfile "mother-ring-03.kicad_sch")
 		(units
 			(unit
@@
 		(property ki_fp_filters "R_*")
 		(sheetname "/")
-		(sheetfile "mother-ring.kicad_sch")
+		(sheetfile "mother-ring-03.kicad_sch")
 		(units
 			(unit
@@
 		(property ki_fp_filters "C_*")
 		(sheetname "/")
-		(sheetfile "mother-ring.kicad_sch")
+		(sheetfile "mother-ring-03.kicad_sch")
 		(units
 			(unit
@@
 		(property ki_fp_filters "Connector*:*_1x??_*")
 		(sheetname "/")
-		(sheetfile "mother-ring.kicad_sch")
+		(sheetfile "mother-ring-03.kicad_sch")
 		(units
 			(unit
@@
 		(property ki_fp_filters "Connector*:*_1x??_*")
 		(sheetname "/")
-		(sheetfile "mother-ring.kicad_sch")
+		(sheetfile "mother-ring-03.kicad_sch")
 		(units
 			(unit
@@
 		(property ki_fp_filters "R_*")
 		(sheetname "/")
-		(sheetfile "mother-ring.kicad_sch")
+		(sheetfile "mother-ring-03.kicad_sch")
 		(units
 			(unit
@@
 		(property ki_fp_filters "C_*")
 		(sheetname "/")
-		(sheetfile "mother-ring.kicad_sch")
+		(sheetfile "mother-ring-03.kicad_sch")
 		(units
 			(unit
@@
 		(property ki_fp_filters "Connector*:*_1x??_*")
 		(sheetname "/")
-		(sheetfile "mother-ring.kicad_sch")
+		(sheetfile "mother-ring-03.kicad_sch")
 		(units
 			(unit
@@
 		(property ki_fp_filters "R_*")
 		(sheetname "/")
-		(sheetfile "mother-ring.kicad_sch")
+		(sheetfile "mother-ring-03.kicad_sch")
 		(units
 			(unit
@@
 		(property ki_fp_filters "Connector*:*_1x??_*")
 		(sheetname "/")
-		(sheetfile "mother-ring.kicad_sch")
+		(sheetfile "mother-ring-03.kicad_sch")
 		(units
 			(unit
@@
 		(property ki_fp_filters "Connector*:*_1x??_*")
 		(sheetname "/")
-		(sheetfile "mother-ring.kicad_sch")
+		(sheetfile "mother-ring-03.kicad_sch")
 		(units
 			(unit
@@
 		(property ki_fp_filters "Connector*:*_1x??_*")
 		(sheetname "/")
-		(sheetfile "mother-ring.kicad_sch")
+		(sheetfile "mother-ring-03.kicad_sch")
 		(units
 			(unit
@@
 		(property ki_fp_filters "Inductor_* L_* *Ferrite*")
 		(sheetname "/")
-		(sheetfile "mother-ring.kicad_sch")
+		(sheetfile "mother-ring-03.kicad_sch")
 		(units
 			(unit
@@
 		(property ki_fp_filters "Connector*:*_1x??_*")
 		(sheetname "/")
-		(sheetfile "mother-ring.kicad_sch")
+		(sheetfile "mother-ring-03.kicad_sch")
 		(units
 			(unit
@@
 		(property ki_fp_filters "Connector*:*_1x??_*")
 		(sheetname "/")
-		(sheetfile "mother-ring.kicad_sch")
+		(sheetfile "mother-ring-03.kicad_sch")
 		(units
 			(unit
@@
 		(property ki_fp_filters "Connector*:*_1x??_*")
 		(sheetname "/")
-		(sheetfile "mother-ring.kicad_sch")
+		(sheetfile "mother-ring-03.kicad_sch")
 		(units
 			(unit
@@
 		(layer "F.SilkS")
 	)
+	(gr_circle
+		(center 0 0)
+		(end 41.25 0)
+		(stroke
+			(width 0.05)
+			(type dot)
+		)
+		(fill no)
+		(layer "F.SilkS")
+	)
 	(gr_line
 		(start 20 -20)
@@
 	)
 	(gr_circle
-		(center -39.652 -11.37)
-		(end -37.952 -11.37)
+		(center -40.27221 -8.928134)
+		(end -38.67221 -8.928134)
 		(stroke
 			(width 0.05)
@@
 	)
 	(gr_circle
-		(center -39.652 11.37)
-		(end -37.952 11.37)
+		(center -40.27221 8.928134)
+		(end -38.67221 8.928134)
+		(stroke
+			(width 0.05)
+			(type solid)
+		)
+		(fill no)
+		(layer "Edge.Cuts")
+	)
+	(gr_circle
+		(center -38.883962 -13.769533)
+		(end -37.283962 -13.769533)
+		(stroke
+			(width 0.05)
+			(type solid)
+		)
+		(fill no)
+		(layer "Edge.Cuts")
+	)
+	(gr_circle
+		(center -38.883962 13.769533)
+		(end -37.283962 13.769533)
 		(stroke
 			(width 0.05)
@@
 	)
 	(gr_circle
-		(center -23.0667 -34.1978)
-		(end -21.3667 -34.1978)
+		(center -25.111409 -32.725825)
+		(end -23.511409 -32.725825)
+		(stroke
+			(width 0.05)
+			(type solid)
+		)
+		(fill no)
+		(layer "Edge.Cuts")
+	)
+	(gr_circle
+		(center -25.111409 32.725825)
+		(end -23.511409 32.725825)
+		(stroke
+			(width 0.05)
+			(type solid)
+		)
+		(fill no)
+		(layer "Edge.Cuts")
+	)
+	(gr_circle
+		(center -20.935957 -35.542203)
+		(end -19.335957 -35.542203)
 		(stroke
 			(width 0.05)
@@
 	)
 	(gr_circle
-		(center -23.0667 34.1978)
-		(end -21.3667 34.1978)
+		(center -20.935957 35.542203)
+		(end -19.335957 35.542203)
 		(stroke
 			(width 0.05)
@@
 	)
 	(gr_circle
-		(center -1.4396 -41.2249)
-		(end 0.2604 -41.2249)
+		(center -3.953637 -41.060093)
+		(end -2.353637 -41.060093)
 		(stroke
 			(width 0.05)
@@
 	)
 	(gr_circle
-		(center -1.4396 41.2249)
-		(end 0.2604 41.2249)
+		(center -3.953637 41.060093)
+		(end -2.353637 41.060093)
 		(stroke
 			(width 0.05)
@@
 		(layer "Edge.Cuts")
 	)
+	(gr_circle
+		(center 1.079799 -41.235865)
+		(end 2.679799 -41.235865)
+		(stroke
+			(width 0.05)
+			(type solid)
+		)
+		(fill no)
+		(layer "Edge.Cuts")
+	)
+	(gr_circle
+		(center 1.079799 41.235865)
+		(end 2.679799 41.235865)
+		(stroke
+			(width 0.05)
+			(type solid)
+		)
+		(fill no)
+		(layer "Edge.Cuts")
+	)
 	(gr_arc
 		(start 14.5 -25.114737)
@@
 		(layer "Edge.Cuts")
 	)
+	(gr_circle
+		(center 23.364257 -33.995205)
+		(end 24.964257 -33.995205)
+		(stroke
+			(width 0.05)
+			(type solid)
+		)
+		(fill no)
+		(layer "Edge.Cuts")
+	)
+	(gr_circle
+		(center 23.364257 33.995205)
+		(end 24.964257 33.995205)
+		(stroke
+			(width 0.05)
+			(type solid)
+		)
+		(fill no)
+		(layer "Edge.Cuts")
+	)
 	(gr_arc
 		(start 25.114737 14.5)
@@
 	)
 	(gr_circle
-		(center 25.396 -32.5054)
-		(end 27.096 -32.5054)
+		(center 27 0)
+		(end 28.4 0)
 		(stroke
 			(width 0.05)
@@
 	)
 	(gr_circle
-		(center 25.396 32.5054)
-		(end 27.096 32.5054)
+		(center 27.333077 -30.894423)
+		(end 28.933077 -30.894423)
 		(stroke
 			(width 0.05)
@@
 	)
 	(gr_circle
-		(center 27 0)
-		(end 28.4 0)
+		(center 27.333077 30.894423)
+		(end 28.933077 30.894423)
 		(stroke
 			(width 0.05)
@@
 	)
 	(gr_circle
-		(center 38.7623 -14.1083)
-		(end 40.4623 -14.1083)
+		(center 37.828701 -16.448387)
+		(end 39.428701 -16.448387)
 		(stroke
 			(width 0.05)
@@
 	)
 	(gr_circle
-		(center 38.7623 14.1083)
-		(end 40.4623 14.1083)
+		(center 37.828701 16.448387)
+		(end 39.428701 16.448387)
+		(stroke
+			(width 0.05)
+			(type solid)
+		)
+		(fill no)
+		(layer "Edge.Cuts")
+	)
+	(gr_circle
+		(center 39.551285 -11.715624)
+		(end 41.151285 -11.715624)
+		(stroke
+			(width 0.05)
+			(type solid)
+		)
+		(fill no)
+		(layer "Edge.Cuts")
+	)
+	(gr_circle
+		(center 39.551285 11.715624)
+		(end 41.151285 11.715624)
 		(stroke
 			(width 0.05)
@@
 	)
 	(segment
-		(start 24.5 13.1)
-		(end 24.5 6.9)
-		(width 0.8)
-		(layer "F.Cu")
-		(net "P+")
-	)
-	(segment
-		(start 24.5 6.9)
-		(end 23.95 6.35)
-		(width 0.8)
-		(layer "F.Cu")
-		(net "P+")
-	)
-	(segment
-		(start 23.95 6.35)
-		(end 22.54 6.35)
-		(width 0.8)
-		(layer "F.Cu")
-		(net "P+")
-	)
-	(segment
-		(start 22 14)
-		(end 23.6 14)
-		(width 0.8)
-		(layer "F.Cu")
-		(net "P+")
-	)
-	(segment
-		(start 23.6 14)
-		(end 24.5 13.1)
-		(width 0.8)
-		(layer "F.Cu")
-		(net "P+")
-	)
-	(segment
 		(start 23.8 12)
 		(end 24.8 11)
@@
 	)
 	(segment
+		(start 24.5 13.1)
+		(end 24.5 6.9)
+		(width 0.8)
+		(layer "F.Cu")
+		(net "P+")
+	)
+	(segment
+		(start 24.5 6.9)
+		(end 23.95 6.35)
+		(width 0.8)
+		(layer "F.Cu")
+		(net "P+")
+	)
+	(segment
+		(start 23.95 6.35)
+		(end 22.54 6.35)
+		(width 0.8)
+		(layer "F.Cu")
+		(net "P+")
+	)
+	(segment
+		(start 22 14)
+		(end 23.6 14)
+		(width 0.8)
+		(layer "F.Cu")
+		(net "P+")
+	)
+	(segment
+		(start 23.6 14)
+		(end 24.5 13.1)
+		(width 0.8)
+		(layer "F.Cu")
+		(net "P+")
+	)
+	(segment
