File: kiban/power-IP2326-MP1584-FPC/power-IP2326-MP1584-FPC.kicad_pcb (KiCad board)
At the start: 2 copper layers, 50 x 40 mm, 23 parts, among them J1 BATTERY, J14 CHARGE, J3 BATTERY, J4 DIRECT, J7 VOUT, J8 VIN, J9 OUTPUT, Q2 AO3401A, U1 MAX16054, U2 TP2326, U3 MP1584EN

Commit message: kiban: power-IP2326-MP1584-FPC regenerate fab outputs + v02/v03 iterations
Parts:
- removed R4: 10kΩ, Resistor_SMD:R_0603_1608Metric
- removed U2: TP2326, neon3:TS2326
- added G***: LOGO, LOGO, B.Cu at (52.1, 52.3)
- added R6: 10kΩ, Resistor_SMD:R_0603_1608Metric, F.Cu at (36.7, 37.2)
- added U5: MP1584EN, neon:MP1584EN, F.Cu at (54.1, 62.9)
- U3: value MP1584EN -> IP2326; footprint neon:MP1584EN -> neon:TS2326
- moved U3 18.0 mm to (56.5, 45.0), turned to 0 degrees
- moved C6 1.07 mm to (36.0, 59.5)
- moved U1 1.00 mm to (36.1, 40.2)
- moved C8 0.76 mm to (39.7, 40.3)
- moved R5 0.18 mm to (39.7, 44.2)
Connections:
- J1 pad 1: P- -> PGND
- J8 pad 2: CHARGE -> POWER
- J8 pad 3: CHARGE -> POWER
- J8 pad 4: P- -> PGND
- U1 pad 3: PGND -> CLR
- U3 pad 1: PGND -> P+
- U3 pad 2: VIN -> BM
- U3 pad 3: VOUT -> PGND
- U3 pad 4: PGND -> CHARGE
Routing:
- net P-: track 63.7 -> 0.00 mm
- net PGND: track 161.8 -> 214.6 mm, vias 20 -> 37
- net POWER: track 41.8 -> 76.4 mm
- net CHARGE: track 28.9 -> 21.0 mm
- net VOUT: track 58.6 -> 62.5 mm
- net GATE: track 8.90 -> 6.27 mm
- net CLR: track 0.00 -> 2.09 mm
- removed copper zone on F.Cu, net P-
Other:
- outline, holes or cut-outs redrawn
- board text added: "BATTERY"
- board text added: "POWER"
