File: kiban/power-IP2326-MP1584-FPC-02/core-M5atom-FPC−02.kicad_sch (KiCad schematic)
At the start: 27 parts, among them J1 BATTERY, J14 CHARGE, J2 BATTERY, J3 BATTERY, J4 DIRECT, J5 LiPo1, J6 LiPo2, J7 VOUT, J8 VIN, J9 OUTPUT, Q2 AO3401A, U1 MAX16054, U2 2S-BMS, U3 IP2326, U5 MP1584EN

Commit message: kiban: power-IP2326-MP1584-FPC regenerate fab outputs + v02/v03 iterations
Parts:
- removed R6: 10kΩ, Resistor_SMD:R_0603_1608Metric, symbol Device:R_Small_US
- added R4: 10kΩ, Resistor_SMD:R_0603_1608Metric, symbol Device:R_Small_US
- U3: footprint neon:TS2326 -> neon3:TS2326
Connections:
- net CLR is gone; now on net PGND: U1.3 (CLR)
- net CHARGE: now also J8.2 (Pin_2), J8.3 (Pin_3)
- net GATE: now also R4.1
- net PGND: no longer J1.1 (Pin_1), J2.1 (Pin_1), J8.4 (Pin_4), U2.5 (P-), U3.3 (B-)
- net POWER: no longer J8.2 (Pin_2), J8.3 (Pin_3)
- net VOUT: now also R4.2
- new net P-: J1.1 (Pin_1), J2.1 (Pin_1), J8.4 (Pin_4), U2.5 (P-), U3.3 (B-)
Other:
- note added: "REMOTE"
- moved on the sheet: C1, C2, C3, FB1, J14, J2, J3, J7, J8, Q2, U3
